Commit message: feat(rl): better parameters for PPO, removed joints limits from model

File: human-robot-rl/models/mate.urdf (robot description, URDF)
Before this commit: robot robot_mate, 8 links, 7 joints
Joints:
- joint q_2: limit lower=-1.57 upper=1.57 effort=100 velocity=100 -> lower=-3.14159 upper=3.14159 effort=100 velocity=100
- joint q_3: limit lower=-1.6 upper=1.6 effort=100 velocity=100 -> lower=-3.14159 upper=3.14159 effort=100 velocity=100
